Commit message: new baseline implementation

File: turtlebot3_description/urdf/simplegoal.urdf (robot description, URDF)
Before this commit: robot simplegoal, 1 links, 0 joints
Links:
- link base_link: geometry collision cylinder length=1 radius=0.01; visual cylinder length=1 radius=0.01

File: turtlebot3_description/urdf/simpleplane.urdf (robot description, URDF)
Before this commit: robot simpleplane, 1 links, 0 joints
Links:
- link base_link: geometry collision box size=200 200 0.01; visual box size=200 200 0.01

Commit message: reward modification

File: turtlebot3_description/urdf/simplegoal.urdf (robot description, URDF)
Before this commit: robot simplegoal, 1 links, 0 joints
Links:
- link base_link: geometry visual cylinder length=1 radius=0.01
