Commit message: PPO training code for orientation with tensorboard logger and modified reward function

File: turtlebot3_description/urdf/turtlebot3_waffle.urdf.xacro (robot description, xacro)
@@ -8,4 +8,11 @@
   <xacro:property name="r200_cam_depth_offset" value="0.01"/>
   <link name="base_footprint"/>
+  <inertial>
+  <mass value="1"/>
+        <inertia ixx="1" ixy="0" ixz="0"
+                iyy="1" iyz="0"
+                izz="1" />
+  </inertial>
+  </link>
   <joint name="base_joint" type="fixed">
     <parent link="base_footprint"/>
