Commit message: Update tm_turtlebot3.urdf

File: Orientation_CW_CCW/turtlebot3_description/urdf/tm_turtlebot3.urdf (robot description, URDF)
Before this commit: robot turtlebot3_burger, 7 links, 6 joints
Links:
- link wheel_left_link: geometry collision cylinder length=0.018 radius=0.04; visual mesh filename=package://turtlebot3_description/meshes/wheels/left_tire.stl scale=0.001 0.001 0.001
